Commit message: before trying to fix gz_sim launch file

File: robot_desc/model/lidar.xacro (robot description, xacro)
@@ -50,5 +50,5 @@
         <topic>scan</topic>
         <!-- check whether it should be gz_frame_id or just frame_id -->
-        <gz_frame_id>laser_frame</gz_frame_id>
+        <!-- <gz_frame_id>laser_frame</gz_frame_id> -->
     </sensor>
 </gazebo>

File: robot_desc/model/robot_core.xacro (robot description, xacro)
@@ -13,5 +13,5 @@
 <xacro:property name= "w_rad" value = "0.1"/>
 <xacro:property name= "w_len" value = "0.05"/>
-<xacro:property name= "w_z" value = "-0.03"/>
+<xacro:property name= "w_z" value = "${2*w_rad-bz_dim/2}"/>
 <!-- constants -->
 <xacro:property name= "pi_const" value = "3.14159265358"/>
@@ -65,5 +65,5 @@
 <parent link = "dummy"/>
 <child link = "body"/>
-<origin rpy= "0 0 0" xyz = "0 0 0"/>
+<origin rpy= "0 0 0" xyz = "0 0 ${w_rad}"/>
 </joint>
 <!-- ############################## -->
@@ -79,4 +79,7 @@
 <origin rpy= "0 0 0" xyz = "0 0 0"/>
 </geometry>
+<material name = "black">
+    <color rgba = "1 1 1 1"/>
+</material>
 </visual>
 <collision>
@@ -103,5 +106,5 @@
 <parent link = "body"/>
 <child link = "LF_wheel"/>
-<origin xyz="${-bx_dim/2 - w_len/2} ${-by_dim/2 + w_rad} ${w_z}" rpy="0 0 0"/>
+<origin xyz="${-bx_dim/2 - w_len/2} ${-by_dim/2 + w_rad} ${bz_dim/2 - w_rad}" rpy="0 0 0"/>
     <axis xyz="1 0 0"/>
     <limit effort="${effort}" velocity="${velocity}"/>
@@ -111,5 +114,5 @@
 <parent link = "body"/>
 <child link = "LB_wheel"/>
-<origin xyz="${-bx_dim/2 - w_len/2 } ${by_dim/2 - w_rad} ${w_z}" rpy="0 0 0"/>
+<origin xyz="${-bx_dim/2 - w_len/2 } ${by_dim/2 - w_rad} ${bz_dim/2 - w_rad}" rpy="0 0 0"/>
     <axis xyz="1 0 0"/>
     <limit effort="${effort}" velocity="${velocity}"/>
@@ -119,5 +122,5 @@
 <parent link = "body"/>
 <child link = "RF_wheel"/>
-<origin xyz="${bx_dim/2 + w_len/2} ${-by_dim/2 + w_rad} ${w_z}" rpy="0 0 0"/>
+<origin xyz="${bx_dim/2 + w_len/2} ${-by_dim/2 + w_rad} ${bz_dim/2 - w_rad}" rpy="0 0 0"/>
     <axis xyz="1 0 0"/>
     <limit effort="${effort}" velocity="${velocity}"/>
@@ -127,5 +130,5 @@
 <parent link = "body"/>
 <child link = "RB_wheel"/>
-<origin xyz="${bx_dim/2 + w_len/2} ${by_dim/2 - w_rad} ${w_z}" rpy="0 0 0"/>
+<origin xyz="${bx_dim/2 + w_len/2} ${by_dim/2 - w_rad} ${bz_dim/2 - w_rad}" rpy="0 0 0"/>
     <axis xyz="1 0 0"/>
     <limit effort="${effort}" velocity="${velocity}"/>

Commit message: before trying to add the camera

File: robot_desc/model/lidar.xacro (robot description, xacro)
@@ -1,5 +1,5 @@
 <?xml version="1.0"?>
 <robot xmlns:xacro="http://www.ros.org/wiki/xacro">
-<xacro:property name = "l_len" value = "0.055"/>
+<xacro:property name = "l_len" value = "0.04"/>
 <xacro:property name = "l_rad" value = ".08"/>
     <joint name="laser_joint" type="fixed">
@@ -32,23 +32,24 @@
 <gazebo reference="laser_frame">
     <sensor name="laser" type="gpu_lidar">
-        <pose> 0 0 0 0 0 0 </pose>
+        <pose>0 0 0 0 0 0</pose>
         <visualize>true</visualize>
         <update_rate>10</update_rate>
         <lidar>
-                <scan>
-                    <horizontal>
-                        <samples>360</samples>
-                        <min_angle>-3.14</min_angle>
-                        <max_angle>3.14</max_angle>
-                    </horizontal>
-                </scan>
-                <range>
-                    <min>0.3</min>
-                    <max>12</max>
-                </range>
+            <scan>
+                <horizontal>
+                    <samples>360</samples>
+                    <resolution>1</resolution>
+                    <min_angle>-3.14159</min_angle>
+                    <max_angle>3.14159</max_angle>
+                </horizontal>
+            </scan>
+            <range>
+                <min>0.3</min>
+                <max>12</max>
+                <resolution>0.01</resolution>
+            </range>
         </lidar>
         <topic>scan</topic>
-        <!-- check whether it should be gz_frame_id or just frame_id -->
-        <frame_id>laser_frame</frame_id>
+        <gz_frame_id>laser_frame</gz_frame_id>
     </sensor>
 </gazebo>

File: robot_desc/model/robot.urdf.xacro (robot description, xacro)
@@ -6,3 +6,9 @@
     <xacro:include filename="$(find robot_desc)/model/robot.gazebo"/>
     <!-- <xacro:include filename="$(find mr_desc)/model/robot_ros2_control.xacro"/> -->
+<gazebo>
+    <plugin filename="gz-sim-sensors-system" name="gz::sim::systems::Sensors">
+        <render_engine>ogre</render_engine>
+        <headless_rendering>true</headless_rendering>        <!-- KEY LINE -->
+    </plugin>
+</gazebo>
 </robot>

File: robot_desc/model/robot_core.xacro (robot description, xacro)
@@ -75,7 +75,7 @@
 <link name = "body">
 <visual>
+<origin rpy= "0 0 0" xyz = "0 0 0"/>
 <geometry>
 <box size = "${bx_dim} ${by_dim} ${bz_dim}"/>
-<origin rpy= "0 0 0" xyz = "0 0 0"/>
 </geometry>
 <material name = "black">
@@ -147,5 +147,5 @@
 <!-- <gazebo >
     <plugin filename="gz-sim-joint-state-publisher-system" name="gz::sim::systems::JointStatePublisher">
-        <topic>joint_states</topic>        <!--from <ros><remapping> -->
+        <topic>joint_states</topic>
         <joint_name>wj_RF</joint_name>
         <joint_name>wj_RB</joint_name>
