Commit message: fix: debug mechanum controller and urdf

File: mecha_robot_desc/model/robot.urdf.xacro (robot description, xacro)
@@ -1,9 +1,10 @@
 <?xml version="1.0"?>
-<robot xmlns:xacro="http://www.ros.org/wiki/xacro" name="robot">
+<robot xmlns:xacro="http://www.ros.org/wiki/xacro"
+    xmlns:gz="http://gazebosim.org/schema" name="robot">
     <xacro:include filename="robot_core.xacro" />
     <!-- <xacro:include filename="gazebo_control.xacro"/> -->
     <xacro:include filename="lidar.xacro" />
     <xacro:include filename="camera.xacro" />
-    <xacro:include filename="$(find robot_desc)/model/robot.gazebo"/>
+    <xacro:include filename="$(find mecha_robot_desc)/model/robot.gazebo"/>
     <!-- <xacro:include filename="$(find mr_desc)/model/robot_ros2_control.xacro"/> -->
     <gazebo>
@@ -13,3 +14,12 @@
         </plugin>
     </gazebo>
+    <gazebo >
+    <plugin filename="gz-sim-joint-state-publisher-system" name="gz::sim::systems::JointStatePublisher">
+        <topic>joint_states</topic>
+        <joint_name>wj_RF</joint_name>
+        <joint_name>wj_RB</joint_name>
+        <joint_name>wj_LF</joint_name>
+        <joint_name>wj_LB</joint_name>
+    </plugin>
+    </gazebo>
 </robot>

File: mecha_robot_desc/model/robot_core.xacro (robot description, xacro)
@@ -5,5 +5,4 @@
 <!-- Date 2026-03-18 -->
 <!-- Updated for Mecanum Drive -->
-<!-- Updated wheels to spheres -->
 <!-- ############################## -->
 <robot name="bob"
@@ -13,6 +12,8 @@
     <xacro:property name="by_dim" value="0.6"/>
     <xacro:property name="bz_dim" value="0.15"/>
-    <!-- Wheel dimensions — only radius needed for a sphere -->
+    <!-- Wheel dimensions -->
     <xacro:property name="w_rad" value="0.1"/>
+    <xacro:property name="w_len" value="0.05"/>
+    <xacro:property name="w_z" value="${2*w_rad - bz_dim/2}"/>
     <!-- Constants -->
     <xacro:property name="pi_const" value="3.14159265358"/>
@@ -22,9 +23,7 @@
     <!-- Masses -->
     <xacro:property name="b_mass" value="${b_dens * bx_dim * by_dim * bz_dim}"/>
-    <!-- Volume of a sphere: (4/3) * pi * r^3 -->
-    <xacro:property name="w_mass" value="${w_dens * (4.0/3.0) * pi_const * w_rad * w_rad * w_rad}"/>
+    <xacro:property name="w_mass" value="${w_dens * pi_const * w_rad * w_rad * w_len}"/>
     <!-- Wheel properties -->
-    <!-- Inertia of a solid sphere: (2/5) * m * r^2 — same for all axes -->
-    <xacro:property name="I_wheel" value="${(2.0/5.0) * w_mass * w_rad * w_rad}"/>
+    <xacro:property name="I_wheel" value="${0.5 * w_mass * w_rad * w_rad}"/>
     <xacro:property name="effort" value="1000"/>
     <xacro:property name="velocity" value="1000"/>
@@ -36,15 +35,15 @@
             <origin rpy="0 0 0" xyz="0 0 0"/>
             <mass value="${w_mass}"/>
-            <!-- Solid sphere: Ixx = Iyy = Izz = (2/5)*m*r^2, all products of inertia = 0 -->
             <inertia ixx="${I_wheel}" ixy="0.0" ixz="0.0" iyy="${I_wheel}" iyz="0.0" izz="${I_wheel}"/>
         </inertial>
     </xacro:macro>
-    <!-- Wheel link macro — no rpy_val needed, spheres are rotationally symmetric -->
-    <xacro:macro name="wheel_def" params="name">
+    <!-- Wheel link macro -->
+    <!-- rpy_val lets each wheel pass in its own roller angle (+45 or -45 deg) -->
+    <xacro:macro name="wheel_def" params="name rpy_val">
         <link name="${name}">
             <visual>
-                <origin rpy="0 0 0" xyz="0 0 0"/>
+                <origin rpy="0 ${rpy_val} 0" xyz="0 0 0"/>
                 <geometry>
-                    <sphere radius="${w_rad}"/>
+                    <cylinder radius="${w_rad}" length="${w_len}"/>
                 </geometry>
                 <material name="black">
@@ -53,7 +52,7 @@
             </visual>
             <collision>
-                <origin rpy="0 0 0" xyz="0 0 0"/>
+                <origin rpy="0 ${rpy_val} 0" xyz="0 0 0"/>
                 <geometry>
-                    <sphere radius="${w_rad}"/>
+                    <cylinder radius="${w_rad}" length="${w_len}"/>
                 </geometry>
             </collision>
@@ -96,11 +95,11 @@
     </link>
     <!-- ############################## -->
-    <!-- Wheel joints -->
+    <!-- Wheel joints — axis is Y for mecanum -->
     <!-- ############################## -->
     <joint name="wj_LF" type="continuous">
         <parent link="body"/>
         <child link="LF_wheel"/>
-        <origin xyz="${-bx_dim/2} ${-by_dim/2 + w_rad} ${bz_dim/2 - w_rad}" rpy="0 0 0"/>
-        <axis xyz="0 1 0"/>
+        <origin xyz="${-bx_dim/2 - w_len/2} ${-by_dim/2 + w_rad} ${bz_dim/2 - w_rad}" rpy="0 0 0"/>
+        <axis xyz="1 0 0"/>
         <limit effort="${effort}" velocity="${velocity}"/>
         <dynamics damping="${damping}" friction="${friction}"/>
@@ -109,6 +108,6 @@
         <parent link="body"/>
         <child link="LB_wheel"/>
-        <origin xyz="${-bx_dim/2} ${by_dim/2 - w_rad} ${bz_dim/2 - w_rad}" rpy="0 0 0"/>
-        <axis xyz="0 1 0"/>
+        <origin xyz="${-bx_dim/2 - w_len/2} ${by_dim/2 - w_rad} ${bz_dim/2 - w_rad}" rpy="0 0 0"/>
+        <axis xyz="1 0 0"/>
         <limit effort="${effort}" velocity="${velocity}"/>
         <dynamics damping="${damping}" friction="${friction}"/>
@@ -117,6 +116,6 @@
         <parent link="body"/>
         <child link="RF_wheel"/>
-        <origin xyz="${bx_dim/2} ${-by_dim/2 + w_rad} ${bz_dim/2 - w_rad}" rpy="0 0 0"/>
-        <axis xyz="0 1 0"/>
+        <origin xyz="${bx_dim/2 + w_len/2} ${-by_dim/2 + w_rad} ${bz_dim/2 - w_rad}" rpy="0 0 0"/>
+        <axis xyz="1 0 0"/>
         <limit effort="${effort}" velocity="${velocity}"/>
         <dynamics damping="${damping}" friction="${friction}"/>
@@ -125,6 +124,6 @@
         <parent link="body"/>
         <child link="RB_wheel"/>
-        <origin xyz="${bx_dim/2 } ${by_dim/2 - w_rad} ${bz_dim/2 - w_rad}" rpy="0 0 0"/>
-        <axis xyz="0 1 0"/>
+        <origin xyz="${bx_dim/2 + w_len/2} ${by_dim/2 - w_rad} ${bz_dim/2 - w_rad}" rpy="0 0 0"/>
+        <axis xyz="1 0 0"/>
         <limit effort="${effort}" velocity="${velocity}"/>
         <dynamics damping="${damping}" friction="${friction}"/>
@@ -132,10 +131,12 @@
     <!-- ############################## -->
     <!-- Wheel links                    -->
-    <!-- Spheres are symmetric — no     -->
-    <!-- rpy_val parameter needed       -->
+    <!-- LF and RB share one diagonal   -->
+    <!-- RF and LB share the other      -->
     <!-- ############################## -->
-    <xacro:wheel_def name="LF_wheel"/>
-    <xacro:wheel_def name="LB_wheel"/>
-    <xacro:wheel_def name="RF_wheel"/>
-    <xacro:wheel_def name="RB_wheel"/>
+    <!-- Left-leaning rollers  (+45 deg) : LF and RB -->
+    <xacro:wheel_def name="LF_wheel" rpy_val="${pi_const/2}"/>
+    <xacro:wheel_def name="RB_wheel" rpy_val="${pi_const/2}"/>
+    <!-- Right-leaning rollers (-45 deg) : RF and LB -->
+    <xacro:wheel_def name="RF_wheel" rpy_val="${-pi_const/2}"/>
+    <xacro:wheel_def name="LB_wheel" rpy_val="${-pi_const/2}"/>
 </robot>
