Commit message: feat: add mecha_robot_desc package

File: mecha_robot_desc/model/lidar.xacro (robot description, xacro)
@@ -1,6 +1,6 @@
 <?xml version="1.0"?>
 <robot xmlns:xacro="http://www.ros.org/wiki/xacro">
-<xacro:property name = "l_len" value = "0.04"/>
-<xacro:property name = "l_rad" value = ".08"/>
+    <xacro:property name = "l_len" value = "0.04"/>
+    <xacro:property name = "l_rad" value = ".08"/>
     <joint name="laser_joint" type="fixed">
         <parent link="body"/>
@@ -30,27 +30,27 @@
         </visual>
     </link>
-<gazebo reference="laser_frame">
-    <sensor name="laser" type="gpu_lidar">
-        <pose>0 0 0 0 0 0</pose>
-        <visualize>true</visualize>
-        <update_rate>10</update_rate>
-        <lidar>
-            <scan>
-                <horizontal>
-                    <samples>360</samples>
-                    <resolution>1</resolution>
-                    <min_angle>-3.14159</min_angle>
-                    <max_angle>3.14159</max_angle>
-                </horizontal>
-            </scan>
-            <range>
-                <min>0.3</min>
-                <max>12</max>
-                <resolution>0.01</resolution>
-            </range>
-        </lidar>
-        <topic>scan</topic>
-        <gz_frame_id>laser_frame</gz_frame_id>
-    </sensor>
-</gazebo>
+    <gazebo reference="laser_frame">
+        <sensor name="laser" type="gpu_lidar">
+            <pose>0 0 0 0 0 0</pose>
+            <visualize>true</visualize>
+            <update_rate>10</update_rate>
+            <lidar>
+                <scan>
+                    <horizontal>
+                        <samples>360</samples>
+                        <resolution>1</resolution>
+                        <min_angle>-3.14159</min_angle>
+                        <max_angle>3.14159</max_angle>
+                    </horizontal>
+                </scan>
+                <range>
+                    <min>0.3</min>
+                    <max>12</max>
+                    <resolution>0.01</resolution>
+                </range>
+            </lidar>
+            <topic>scan</topic>
+            <gz_frame_id>laser_frame</gz_frame_id>
+        </sensor>
+    </gazebo>
 </robot>

File: mecha_robot_desc/model/robot.urdf.xacro (robot description, xacro)
@@ -7,9 +7,9 @@
     <xacro:include filename="$(find robot_desc)/model/robot.gazebo"/>
     <!-- <xacro:include filename="$(find mr_desc)/model/robot_ros2_control.xacro"/> -->
-<gazebo>
-    <plugin filename="gz-sim-sensors-system" name="gz::sim::systems::Sensors">
-        <render_engine>ogre</render_engine>
-        <headless_rendering>true</headless_rendering>        <!-- KEY LINE -->
-    </plugin>
-</gazebo>
+    <gazebo>
+        <plugin filename="gz-sim-sensors-system" name="gz::sim::systems::Sensors">
+            <render_engine>ogre</render_engine>
+            <headless_rendering>true</headless_rendering>
+        </plugin>
+    </gazebo>
 </robot>

Commit message: before trying to fix the launch file

File: mecha_robot_desc/model/lidar.xacro (robot description, xacro)
@@ -2,5 +2,5 @@
 <robot xmlns:xacro="http://www.ros.org/wiki/xacro">
     <xacro:property name = "l_len" value = "0.04"/>
-    <xacro:property name = "l_rad" value = ".08"/>
+    <xacro:property name = "l_rad" value = ".04"/>
     <joint name="laser_joint" type="fixed">
         <parent link="body"/>

File: mecha_robot_desc/model/robot_core.xacro (robot description, xacro)
@@ -9,9 +9,9 @@
     xmlns:xacro="http://www.ros.org/wiki/xacro">
     <!-- dimensions of the body -->
-    <xacro:property name="bx_dim" value="0.4"/>
-    <xacro:property name="by_dim" value="0.6"/>
-    <xacro:property name="bz_dim" value="0.15"/>
+    <xacro:property name="bx_dim" value="0.1"/>
+    <xacro:property name="by_dim" value="0.3"/>
+    <xacro:property name="bz_dim" value="0.08"/>
     <!-- Wheel dimensions -->
-    <xacro:property name="w_rad" value="0.1"/>
+    <xacro:property name="w_rad" value="0.07"/>
     <xacro:property name="w_len" value="0.05"/>
     <xacro:property name="w_z" value="${2*w_rad - bz_dim/2}"/>
@@ -19,6 +19,6 @@
     <xacro:property name="pi_const" value="3.14159265358"/>
     <!-- Densities -->
-    <xacro:property name="b_dens" value="1"/>
-    <xacro:property name="w_dens" value="1"/>
+    <xacro:property name="b_dens" value="10000"/>
+    <xacro:property name="w_dens" value="10000"/>
     <!-- Masses -->
     <xacro:property name="b_mass" value="${b_dens * bx_dim * by_dim * bz_dim}"/>
